Commit message: A10 P1 1h17min

File: Parte11/psr_parte11_p1/urdf/scara.urdf (robot description, URDF)
Before this commit: robot myscara, 2 links, 1 joints
Joints:
- joint base_link_to_link1: limit (none) -> lower=0.0 upper=6.28 effort=1000.0 velocity=0.5

Commit message: A10 P1 1h22min

File: Parte11/psr_parte11_p1/urdf/scara.urdf (robot description, URDF)
Before this commit: robot myscara, 2 links, 1 joints
Links:
- added link link1b; visual cylinder length=0.6 radius=0.3
- link base_link: geometry visual cylinder length=0.6 radius=0.3
Joints:
- added joint link1_to_link1b: type fixed, parent link1, child link1b, origin xyz=0 0 -0.3 rpy=0 0 0

Commit message: A10 P1 1h30min

File: Parte11/psr_parte11_p1/urdf/scara.urdf (robot description, URDF)
Before this commit: robot myscara, 3 links, 2 joints
Links:
- added link link2; visual box size=3.0 0.6 0.6
- added link link2b; visual cylinder length=0.6 radius=0.3
- added link link2c; visual cylinder length=0.6 radius=0.3
- added link link3; visual cylinder length=2 radius=0.15
Joints:
- added joint link1_to_link2: type revolute, parent link1, child link2, origin xyz=3 0 0 rpy=0 0 0, axis 0 0 1, limit lower=0.0 upper=6.28 effort=1000.0 velocity=0.5
- added joint link1_to_link2b: type fixed, parent link1, child link2b, origin xyz=3 0 -0.3 rpy=0 0 0
- added joint link2_to_link2c: type fixed, parent link2, child link2c, origin xyz=3 0 -0.3 rpy=0 0 0
- added joint link2c_to_link3: type prismatic, parent link2c, child link3, origin xyz=0 0 0 rpy=0 0 0, axis 0 0 1, limit lower=-0.5 upper=0 effort=1000.0 velocity=0.5
